File: ESP32-S2/_autosave-ESP32-S2.kicad_pcb (KiCad board)
At the start: 2 copper layers, 27.9 x 70 mm, 39 parts, among them J1 Conn_01x18_Male, J2 Conn_01x21_Male, J3 USB_A, J4 TYPE-C-31-M-12, Q2 L8050QLT1G, Q3 L8050QLT1G, SW1 EN/RESET, SW2 BOOT/SELECT, U2 ESP32-S2-WROOM-ESP32-S2-WROOM, U3 AMS1117-3.3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

Commit message: Test Routing Done
Parts:
- moved SW2 0.39 mm to (159.2, 119.5)
Routing:
- net GND: track 174.1 -> 173.5 mm
Changed lines of the file:
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@@
   )
   (module Button_Switch_SMD:SW_SPST_CK_KXT3 (layer F.Cu)
-    (at 158.775 119.55)
+    (at 159.165 119.54)
     (descr https://www.ckswitches.com/media/1465/kxt3.pdf)
     (tags "Switch SPST KXT3")
@@
   (segment (start 161.98 122.85) (end 160.825 122.85) (width 0.4) (layer F.Cu) (net 1))
   (segment (start 163.725 124.595) (end 161.98 122.85) (width 0.4) (layer F.Cu) (net 1))
-  (segment (start 160.825 119.975) (end 160.4 119.55) (width 0.4) (layer F.Cu) (net 1))
   (segment (start 160.825 122.85) (end 160.825 119.975) (width 0.4) (layer F.Cu) (net 1))
   (segment (start 153.505 126.88) (end 152.075 125.45) (width 0.4) (layer F.Cu) (net 1))
@@
   (segment (start 157.15 69.76) (end 159.39 69.76) (width 0.2) (layer F.Cu) (net 3))
   (segment (start 152.135 115.94) (end 155.2 115.94) (width 0.2) (layer F.Cu) (net 4))
-  (segment (start 157.15 117.89) (end 157.15 119.55) (width 0.2) (layer F.Cu) (net 4))
   (via (at 151.77 120.22) (size 0.8) (drill 0.4) (layers F.Cu B.Cu) (net 4))
   (segment (start 150.39 121.6) (end 151.77 120.22) (width 0.2) (layer F.Cu) (net 4))
@@
   (segment (start 155.46 116.2) (end 157.15 117.89) (width 0.2) (layer F.Cu) (net 4))
   (segment (start 155.2 115.94) (end 155.46 116.2) (width 0.2) (layer F.Cu) (net 4))
+  (segment (start 157.15 119.15) (end 157.54 119.54) (width 0.2) (layer F.Cu) (net 4))
+  (segment (start 157.15 117.89) (end 157.15 119.15) (width 0.2) (layer F.Cu) (net 4))
   (segment (start 148.875 100.585) (end 148.61 100.85) (width 0.2) (layer F.Cu) (net 5))
   (segment (start 148.875 98.025) (end 148.875 100.585) (width 0.2) (layer F.Cu) (net 5))
