File: ESP32-S2/ESP32-S2.sch (KiCad schematic (older format))
At the start: 50 parts, among them IC1 IP4220CZ6, J1 USB_A, J2 TYPE-C-31-M-12, J3 Conn_01x18_Male, J4 S2B-PH-SM4-TB(LF)(SN), J5 Conn_01x22_Male, Q1 L8050QLT1G, Q2 L8050QLT1G, SW1 SW_Push, SW2 SW_Push, U1 ESP32-S2-WROOM-ESP32-S2-WROOM, U2 MCP73831-2-OT, U3 AMS1117-3.3, U4 CH340C

Commit message: Minor changes
Parts:
- R10, R9: value 100 -> 100k
Connections:
- net labels removed: VDD33, VIO
Other:
- note added: "Connect 4.2 rated 1C Lithium\nPolymer Battery"
- note removed: "Connect 4.2 rated 1C Lithium\nPolymer Battery - 300 mAh"
Changed lines of the file:
@@
 Text Label 6150 1515 2    50   ~ 0
 GPIO42
-Text Label 3390 3185 2    50   ~ 0
-VDD33
 Wire Wire Line
 	4810 6835 5020 6835
@@
 Wire Notes Line
 	3705 715  470  715
-Text Label 675  1230 0    50   ~ 0
-VDD33
-Wire Wire Line
-	675  1230 1000 1230
 Wire Wire Line
 	1000 1130 675  1130
@@
 VBUSA
 Text Label 6660 2625 0    50   ~ 0
-VIO
+VI
 $Comp
 L Device:C C7
@@
 $EndComp
 Text Label 5245 2750 2    50   ~ 0
-VBUSA
+VI
 Wire Wire Line
 	4905 2750 5245 2750
@@
 Text Label 3980 1060 2    50   ~ 0
 GPIO15
-$Comp
-L power:+3.3V #PWR014
-U 1 1 610BFFB6
-P 5125 1150
-F 0 "#PWR014" H 5125 1000 50  0001 C CNN
-F 1 "+3.3V" H 5140 1323 50  0000 C CNN
-F 2 "" H 5125 1150 50  0001 C CNN
-F 3 "" H 5125 1150 50  0001 C CNN
-	1    5125 1150
-	0    1    1    0
-$EndComp
 Wire Wire Line
 	4905 1150 5125 1150
@@
 GPIO16
 Text Label 10080 5385 0    50   ~ 0
-VIO
+VI
 $Comp
 L power:GND #PWR025
@@
 P 4675 4980
 F 0 "R10" H 4745 5026 50  0000 L CNN
-F 1 "100" H 4745 4935 50  0000 L CNN
+F 1 "100k" H 4745 4935 50  0000 L CNN
 F 2 "Resistor_SMD:R_0603_1608Metric" V 4605 4980 50  0001 C CNN
 F 3 "~" H 4675 4980 50  0001 C CNN
@@
 P 4675 4500
 F 0 "R9" H 4745 4546 50  0000 L CNN
-F 1 "100" H 4745 4455 50  0000 L CNN
+F 1 "100k" H 4745 4455 50  0000 L CNN
 F 2 "Resistor_SMD:R_0603_1608Metric" V 4605 4500 50  0001 C CNN
 F 3 "~" H 4675 4500 50  0001 C CNN
@@
 Wire Wire Line
 	4675 4745 4675 4650
-Text Notes 5170 4300 0    50   ~ 0
-Connect 4.2 rated 1C Lithium\nPolymer Battery - 300 mAh
 Text Notes 5990 5585 0    50   ~ 0
 I_charge = 1/R_prog\nI_charge = 1/4700 \nI_charge = 213 mA\n \nwhere:\nR_prog is in Ohms\nI_charge is in mA
@@
 Wire Notes Line
 	6980 5930 6980 5925
+Text Notes 5170 4300 0    50   ~ 0
+Connect 4.2 rated 1C Lithium\nPolymer Battery
+$Comp
+L power:+3.3V #PWR014
+U 1 1 610BFFB6
+P 770 1230
+F 0 "#PWR014" H 770 1080 50  0001 C CNN
+F 1 "+3.3V" H 785 1403 50  0000 C CNN
+F 2 "" H 770 1230 50  0001 C CNN
+F 3 "" H 770 1230 50  0001 C CNN
+	1    770  1230
+	0    -1   -1   0
+$EndComp
+Wire Wire Line
+	770  1230 1000 1230
+$Comp
+L power:+3.3V #PWR?
+U 1 1 60AF9A04
+P 5125 1150
+F 0 "#PWR?" H 5125 1000 50  0001 C CNN
+F 1 "+3.3V" H 5140 1323 50  0000 C CNN
+F 2 "" H 5125 1150 50  0001 C CNN
+F 3 "" H 5125 1150 50  0001 C CNN
+	1    5125 1150
+	0    1    1    0
+$EndComp
 $EndSCHEMATC

Commit message: Changed Neopixel
Parts:
- removed C11: 0.1uF, Capacitor_SMD:C_0603_1608Metric, symbol Device:C_Small
- removed D6: Inolux_IN-PI554FCH, LED_SMD:LED_Inolux_IN-PI554FCH_PLCC4_5.0x5.0mm_P3.2mm, symbol LED:Inolux_IN-PI554FCH
- added D6: WS2812B, WS2018:WS2812B2020, symbol LED:WS2812B
Connections:
- wire segments 264 -> 262
Changed lines of the file:
@@
 Wire Notes Line
 	9220 3155 11330 3155
-$Comp
-L LED:Inolux_IN-PI554FCH D6
-U 1 1 60BE62B2
-P 10080 5685
-F 0 "D6" H 10424 5731 50  0000 L CNN
-F 1 "Inolux_IN-PI554FCH" H 10424 5640 50  0000 L CNN
-F 2 "LED_SMD:LED_Inolux_IN-PI554FCH_PLCC4_5.0x5.0mm_P3.2mm" H 10130 5385 50  0001 L TNN
-F 3 "http://www.inolux-corp.com/datasheet/SMDLED/Addressable%20LED/IN-PI554FCH.pdf" H 10180 5310 50  0001 L TNN
-	1    10080 5685
-	1    0    0    -1
-$EndComp
 Text Label 9615 5685 1    50   ~ 0
 GPIO16
@@
 	1    0    0    -1
 $EndComp
-Wire Wire Line
-	10080 5985 10080 6045
-$Comp
-L Device:C_Small C11
-U 1 1 60C72A58
-P 9690 5890
-F 0 "C11" H 9782 5936 50  0000 L CNN
-F 1 "0.1uF" H 9782 5845 50  0000 L CNN
-F 2 "Capacitor_SMD:C_0603_1608Metric" H 9690 5890 50  0001 C CNN
-F 3 "~" H 9690 5890 50  0001 C CNN
-	1    9690 5890
-	1    0    0    -1
-$EndComp
-Wire Wire Line
-	9690 5790 9690 5685
-Wire Wire Line
-	9615 5685 9690 5685
-Connection ~ 9690 5685
-Wire Wire Line
-	9690 5685 9780 5685
-Wire Wire Line
-	9690 5990 9690 6045
-Wire Wire Line
-	9690 6045 10080 6045
-Connection ~ 10080 6045
-Wire Wire Line
-	10080 6045 10080 6055
 $Comp
 L Device:R_Small R16
@@
 $EndComp
 Wire Wire Line
-	10385 5790 10385 5685
-Wire Wire Line
 	10385 5685 10380 5685
 Wire Wire Line
 	10385 5990 10385 6045
-Wire Wire Line
-	10385 6045 10080 6045
 $Comp
 L Diode:1N5819 D3
@@
 	770  1230 1000 1230
 $Comp
-L power:+3.3V #PWR?
+L power:+3.3V #PWR028
 U 1 1 60AF9A04
 P 5125 1150
-F 0 "#PWR?" H 5125 1000 50  0001 C CNN
+F 0 "#PWR028" H 5125 1000 50  0001 C CNN
 F 1 "+3.3V" H 5140 1323 50  0000 C CNN
 F 2 "" H 5125 1150 50  0001 C CNN
@@
 	0    1    1    0
 $EndComp
+$Comp
+L LED:WS2812B D6
+U 1 1 609FC678
+P 10080 5685
+F 0 "D6" H 10424 5731 50  0000 L CNN
+F 1 "WS2812B" H 10424 5640 50  0000 L CNN
+F 2 "WS2018:WS2812B2020" H 10130 5385 50  0001 L TNN
+F 3 "https://cdn-shop.adafruit.com/datasheets/WS2812B.pdf" H 10180 5310 50  0001 L TNN
+	1    10080 5685
+	1    0    0    -1
+$EndComp
+Wire Wire Line
+	10385 5790 10385 5685
+Wire Wire Line
+	9615 5685 9780 5685
+Wire Wire Line
+	10080 5985 10080 6040
+Wire Wire Line
+	10385 6045 10085 6045
+Wire Wire Line
+	10085 6045 10085 6040
+Wire Wire Line
+	10085 6040 10080 6040
+Connection ~ 10080 6040
+Wire Wire Line
+	10080 6040 10080 6055
 $EndSCHEMATC

Commit message: replaces L8050QLT1G with MMBT8050
Parts:
- removed Q1, Q2: L8050QLT1G, L8050QLT1G:L8050QLT1G, symbol Device:Q_NPN_BCE
- added U2, U3: MMBT8050, MMBT8050:MMBT8050, symbol MMBT8050:MMBT8050
- J1: symbol Connector:USB_A -> ESP32-S2-rescue:USB_A-Connector
- U6: renamed from U4; symbol Interface_USB:CH340C -> ESP32-S2-rescue:CH340C-Interface_USB
- renumbered C9 to C10, C10 to C11, C13 to C9, U2 to U4, U3 to U5

Commit message: Updated schematics
Parts:
- removed D1, D2: LED, LED_SMD:LED_0603_1608Metric_Castellated, symbol Device:LED
- removed R6, R7: 1k, Resistor_SMD:R_0603_1608Metric, symbol Device:R
- renumbered D3 to D1, D4 to D2, D5 to D3
Other:
- moved on the sheet: C2, C3
Changed lines of the file:
@@
 GPIO0
 Wire Wire Line
-	3930 2985 3970 2985
-Wire Wire Line
-	3390 3185 3630 3185
-Wire Wire Line
-	3390 2975 3390 3185
-Wire Wire Line
-	3630 3185 3630 3385
-Connection ~ 3630 3185
-Wire Wire Line
-	3630 2985 3630 3185
+	3830 1985 3870 1985
+Wire Wire Line
+	3290 2185 3530 2185
+Wire Wire Line
+	3290 1975 3290 2185
+Wire Wire Line
+	3530 2185 3530 2385
+Connection ~ 3530 2185
+Wire Wire Line
+	3530 1985 3530 2185
 $Comp
 L power:+3.3V #PWR06
 U 1 1 6005C874
-P 3390 2975
-F 0 "#PWR06" H 3390 2825 50  0001 C CNN
-F 1 "+3.3V" H 3405 3148 50  0000 C CNN
-F 2 "" H 3390 2975 50  0001 C CNN
-F 3 "" H 3390 2975 50  0001 C CNN
-	1    3390 2975
+P 3290 1975
+F 0 "#PWR06" H 3290 1825 50  0001 C CNN
+F 1 "+3.3V" H 3305 2148 50  0000 C CNN
+F 2 "" H 3290 1975 50  0001 C CNN
+F 3 "" H 3290 1975 50  0001 C CNN
+	1    3290 1975
 	1    0    0    -1
 $EndComp
@@
 L Device:C C2
 U 1 1 60022F39
-P 3780 2985
-F 0 "C2" V 3910 2935 50  0000 L CNN
-F 1 "0.1uF" V 3640 2885 50  0000 L CNN
-F 2 "Capacitor_SMD:C_0603_1608Metric" H 3818 2835 50  0001 C CNN
-F 3 "~" H 3780 2985 50  0001 C CNN
-	1    3780 2985
+P 3680 1985
+F 0 "C2" V 3810 1935 50  0000 L CNN
+F 1 "0.1uF" V 3540 1885 50  0000 L CNN
+F 2 "Capacitor_SMD:C_0603_1608Metric" H 3718 1835 50  0001 C CNN
+F 3 "~" H 3680 1985 50  0001 C CNN
+	1    3680 1985
 	0    -1   -1   0
 $EndComp
@@
 L Device:C C3
 U 1 1 60021E18
-P 3780 3385
-F 0 "C3" V 3910 3335 50  0000 L CNN
-F 1 "10uF" V 3630 3295 50  0000 L CNN
-F 2 "Capacitor_SMD:C_0603_1608Metric" H 3818 3235 50  0001 C CNN
-F 3 "~" H 3780 3385 50  0001 C CNN
-	1    3780 3385
+P 3680 2385
+F 0 "C3" V 3810 2335 50  0000 L CNN
+F 1 "10uF" V 3530 2295 50  0000 L CNN
+F 2 "Capacitor_SMD:C_0603_1608Metric" H 3718 2235 50  0001 C CNN
+F 3 "~" H 3680 2385 50  0001 C CNN
+	1    3680 2385
 	0    -1   -1   0
 $EndComp
@@
 	430  4055 430  4080
 Wire Wire Line
-	3970 2985 3970 3185
+	3870 1985 3870 2185
 $Comp
 L power:GND #PWR09
 U 1 1 600B09CA
-P 4065 3245
-F 0 "#PWR09" H 4065 2995 50  0001 C CNN
-F 1 "GND" H 4070 3072 50  0000 C CNN
-F 2 "" H 4065 3245 50  0001 C CNN
-F 3 "" H 4065 3245 50  0001 C CNN
-	1    4065 3245
-	1    0    0    -1
-$EndComp
-Wire Wire Line
-	4065 3185 3970 3185
-Connection ~ 3970 3185
-Wire Wire Line
-	3970 3185 3970 3385
+P 3965 2245
+F 0 "#PWR09" H 3965 1995 50  0001 C CNN
+F 1 "GND" H 3970 2072 50  0000 C CNN
+F 2 "" H 3965 2245 50  0001 C CNN
+F 3 "" H 3965 2245 50  0001 C CNN
+	1    3965 2245
+	1    0    0    -1
+$EndComp
+Wire Wire Line
+	3965 2185 3870 2185
+Connection ~ 3870 2185
+Wire Wire Line
+	3870 2185 3870 2385
 Wire Wire Line
 	2200 3530 2335 3530
@@
 	1000 3630 895  3630
 Wire Wire Line
-	4065 3185 4065 3245
+	3965 2185 3965 2245
 Text Label 895  3630 2    50   ~ 0
 GND
@@
 $EndComp
 Wire Wire Line
-	3930 3385 3970 3385
+	3830 2385 3870 2385
 Wire Wire Line
 	8945 3090 8945 3000
@@
 Connection ~ 8290 2625
 $Comp
-L Device:LED D4
+L Device:LED D2
 U 1 1 602D9272
 P 8770 2625
-F 0 "D4" H 8809 2507 50  0000 R CNN
+F 0 "D2" H 8809 2507 50  0000 R CNN
 F 1 "LED" H 8835 2720 50  0000 R CNN
 F 2 "LED_SMD:LED_0603_1608Metric_Castellated" H 8770 2625 50  0001 C CNN
@@
 	5875 2915 6230 2915
 $Comp
-L Device:R R6
-U 1 1 60104A04
-P 3630 1210
-F 0 "R6" H 3700 1256 50  0000 L CNN
-F 1 "1k" H 3700 1165 50  0000 L CNN
-F 2 "Resistor_SMD:R_0603_1608Metric" V 3560 1210 50  0001 C CNN
-F 3 "~" H 3630 1210 50  0001 C CNN
-	1    3630 1210
-	1    0    0    -1
-$EndComp
-$Comp
-L Device:R R7
-U 1 1 60104F07
-P 3980 1210
-F 0 "R7" H 4050 1256 50  0000 L CNN
-F 1 "1k" H 4050 1165 50  0000 L CNN
-F 2 "Resistor_SMD:R_0603_1608Metric" V 3910 1210 50  0001 C CNN
-F 3 "~" H 3980 1210 50  0001 C CNN
-	1    3980 1210
-	1    0    0    -1
-$EndComp
-$Comp
 L Device:C C11
 U 1 1 60DF3BEA
@@
 	10420 1085 10420 985
 Wire Wire Line
-	3630 1660 3630 1860
-$Comp
-L Device:LED D2
-U 1 1 60106F43
-P 3980 1510
-F 0 "D2" V 4030 1370 50  0000 C CNN
-F 1 "LED" V 3950 1355 50  0000 C CNN
-F 2 "LED_SMD:LED_0603_1608Metric_Castellated" H 3980 1510 50  0001 C CNN
-F 3 "~" H 3980 1510 50  0001 C CNN
-	1    3980 1510
-	0    -1   -1   0
-$EndComp
-$Comp
-L Device:LED D1
-U 1 1 60106194
-P 3630 1510
-F 0 "D1" V 3680 1390 50  0000 C CNN
-F 1 "LED" V 3600 1365 50  0000 C CNN
-F 2 "LED_SMD:LED_0603_1608Metric_Castellated" H 3630 1510 50  0001 C CNN
-F 3 "~" H 3630 1510 50  0001 C CNN
-	1    3630 1510
-	0    -1   -1   0
-$EndComp
-$Comp
-L power:GND #PWR07
-U 1 1 60E56461
-P 3835 1875
-F 0 "#PWR07" H 3835 1625 50  0001 C CNN
-F 1 "GND" H 3840 1702 50  0000 C CNN
-F 2 "" H 3835 1875 50  0001 C CNN
-F 3 "" H 3835 1875 50  0001 C CNN
-	1    3835 1875
-	1    0    0    -1
-$EndComp
-Wire Wire Line
-	3630 1860 3835 1860
-Wire Wire Line
-	3835 1860 3835 1875
-Wire Wire Line
-	3835 1860 3980 1860
-Wire Wire Line
-	3980 1660 3980 1860
-Connection ~ 3835 1860
-Text Label 3630 1060 2    50   ~ 0
-GPIO14
-Wire Wire Line
 	10820 1635 11085 1635
 Wire Wire Line
@@
 Wire Wire Line
 	10820 2335 11085 2335
-Text Label 3980 1060 2    50   ~ 0
-GPIO15
 Wire Wire Line
 	4905 1150 5125 1150
@@
 	3015 715  3015 3850
 Wire Notes Line
-	3015 2380 4525 2380
-Wire Notes Line
 	4525 2380 4525 2385
 $Comp
@@
 	10385 5990 10385 6045
 $Comp
-L Diode:1N5819 D3
+L Diode:1N5819 D1
 U 1 1 60956142
 P 7725 1320
-F 0 "D3" H 7725 1103 50  0000 C CNN
+F 0 "D1" H 7725 1103 50  0000 C CNN
 F 1 "1N5819" H 7725 1194 50  0000 C CNN
 F 2 "Diode_SMD:D_1206_3216Metric" H 7725 1145 50  0001 C CNN
@@
 $EndComp
 $Comp
-L Device:LED D5
+L Device:LED D3
 U 1 1 60A5A83D
 P 8930 4815
-F 0 "D5" H 8923 5032 50  0000 C CNN
+F 0 "D3" H 8923 5032 50  0000 C CNN
 F 1 "LED" H 8923 4941 50  0000 C CNN
 F 2 "LED_SMD:LED_0603_1608Metric_Castellated" H 8930 4815 50  0001 C CNN
