File: ESP32-S2/ESP32-S2.kicad_pcb (KiCad board)
At the start: 4 copper layers, 27.8 x 70.3 mm, 45 parts, among them IC1 IP4220CZ6, J1 USB_A, J2 TYPE-C-31-M-12, J3 Conn_01x18_Male, J4 S2B-PH-SM4-TB(LF)(SN), J5 Conn_01x22_Male, SW1 SW_Push, SW2 SW_Push, U1 ESP32-S2-WROOM-ESP32-S2-WROOM, U2 MMBT8050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

Commit message: Changes in Routing
Parts:
- moved R2 4.59 mm to (151.9, 106.3)
- moved R11 1.68 mm to (152.0, 108.5)
- moved C12 1.26 mm to (155.9, 108.6)
- moved C9 1.17 mm to (154.1, 104.0)
- moved R12 1.17 mm to (151.0, 104.0)
- moved C11 0.80 mm to (157.2, 104.0), turned to 0 degrees
- moved R8 0.38 mm to (144.3, 103.0)
- moved R10 0.33 mm to (147.9, 101.9)
- moved R7 0.23 mm to (142.3, 103.0)
Routing:
- net +3V3: track 36.0 -> 48.8 mm
- net /GPIO18: track 34.8 -> 28.1 mm
- net Net-(C9-Pad1): track 36.1 -> 32.9 mm, vias 4 -> 2
- net /VI: track 86.6 -> 84.0 mm
- net /GPIO8: track 45.7 -> 43.9 mm
- net /CHIP_PU: track 89.1 -> 87.5 mm, vias 6 -> 5
- net Net-(D3-Pad1): track 38.9 -> 37.3 mm
- net /GPIO0: track 60.2 -> 59.5 mm
- net Net-(R11-Pad1): track 26.0 -> 26.7 mm, vias 4 -> 2
- net /GPIO10: track 18.8 -> 18.1 mm
- net Net-(C12-Pad1): track 6.50 -> 7.09 mm
- net /DN1: track 36.4 -> 36.9 mm
- net /GPIO15: track 22.0 -> 22.5 mm
- net GND: track 123.3 -> 123.8 mm, vias 27 -> 28

Commit message: added minor routing changes
Routing:
- net +3V3: track 48.8 -> 47.3 mm
- net /GPIO18: track 28.1 -> 27.0 mm
- net /CHIP_PU: track 87.5 -> 86.4 mm

Commit message: Minor Changes
Parts:
- moved F1 0.43 mm to (159.2, 118.4)
- moved D1 0.10 mm to (159.0, 122.2)
- moved IC1 0.08 mm to (158.9, 113.4)
Routing:
- net Net-(D3-Pad1): track 37.6 -> 24.8 mm
- net /DN1: track 36.9 -> 35.2 mm
- net /GPIO26: track 20.0 -> 18.9 mm
- net /GPIO0: track 59.5 -> 58.4 mm
- net GND: track 123.7 -> 123.0 mm
- net /GPIO36: track 15.0 -> 15.7 mm
- net Net-(R11-Pad1): track 27.0 -> 27.7 mm
- net /GPIO34: track 17.4 -> 16.8 mm
- net /GPIO35: track 16.3 -> 16.8 mm
- net /CHIP_PU: track 86.4 -> 85.8 mm
- net /~RTS: track 14.4 -> 13.8 mm
- net /GPIO20: track 51.8 -> 51.7 mm, vias 2 -> 3

Commit message: Optimised 4-lyr routing v.4lyr.2
Parts:
- moved R7 22.4 mm to (149.9, 124.0), turned to 180 degrees
- moved R8 21.1 mm to (146.8, 124.0), turned to 180 degrees
- moved C9 16.4 mm to (151.0, 120.1), turned to 270 degrees
- moved R12 16.2 mm to (149.3, 120.1), turned to 90 degrees
- moved IC1 14.6 mm to (146.3, 120.8)
- moved D4 13.8 mm to (157.3, 105.2), turned to 0 degrees
- moved R1 13.2 mm to (149.7, 94.8)
- moved R9 12.8 mm to (156.6, 113.4), turned to 90 degrees
- moved R11 10.9 mm to (153.6, 119.3), turned to 180 degrees
- moved R2 10.1 mm to (142.4, 109.5), turned to 0 degrees
- moved R10 7.95 mm to (142.4, 107.6), turned to 180 degrees
- moved R14 7.77 mm to (154.1, 105.1)
- moved R5 6.99 mm to (150.8, 116.6), turned to 270 degrees
- moved U4 6.22 mm to (153.9, 122.1), turned to 0 degrees
- moved C11 5.95 mm to (156.6, 109.9), turned to 90 degrees
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Connections:
- J3 pad 18: /VI -> /GPIO16
- J5 pad 22: /GPIO16 -> /VI
Routing:
- net GND: track 123.0 -> 75.5 mm, vias 28 -> 34
- net /VI: track 84.1 -> 53.9 mm
- net Net-(C9-Pad1): track 32.9 -> 4.51 mm, vias 2 -> 0
- net Net-(R11-Pad1): track 27.7 -> 2.00 mm, vias 2 -> 0
- net +BATT: track 30.5 -> 6.58 mm, vias 3 -> 0
- net Net-(D3-Pad1): track 24.8 -> 1.52 mm, vias 2 -> 0
- net /GPIO16: track 63.4 -> 40.6 mm, vias 2 -> 0
- net /GPIO18: track 27.0 -> 4.31 mm, vias 4 -> 2
- net /CHIP_PU: track 85.8 -> 66.2 mm, vias 5 -> 2
- net /GPIO0: track 58.4 -> 75.7 mm, vias 4 -> 2
- net /GPIO8: track 43.9 -> 61.0 mm, vias 3 -> 2
- net /TXD0: track 63.3 -> 47.6 mm
- net /RXD0: track 61.7 -> 46.5 mm, vias 1 -> 2
- net /GPIO19: track 54.3 -> 63.6 mm, vias 3 -> 1
- net +3V3: track 47.6 -> 39.5 mm, vias 5 -> 7
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Other:
- board text removed: "Designed By: 1. Dhairya 2. Chaitravi 3. Sakshi 4. Vedant 5. Omkar"

Commit message: Routing Optimizations
Parts:
- moved C12 3.80 mm to (147.5, 104.9), turned to 180 degrees
- moved R14 2.22 mm to (151.9, 104.9), turned to 180 degrees
Routing:
- net GND: track 75.5 -> 72.1 mm, vias 34 -> 36
- net /GPIO8: track 61.0 -> 63.4 mm
- net /GPIO34: track 18.5 -> 16.6 mm
- net /GPIO11: track 16.4 -> 14.6 mm
- net Net-(C12-Pad1): track 2.84 -> 4.57 mm
- net Net-(D4-Pad2): track 5.97 -> 7.53 mm
- net /GPIO16: track 40.6 -> 41.7 mm
- net /VI: track 53.9 -> 54.9 mm
- net /VBUSA: track 13.7 -> 13.1 mm
- net /GPIO37: track 15.7 -> 16.2 mm
- net /GPIO35: track 17.7 -> 18.2 mm
- net /GPIO20: track 58.7 -> 59.0 mm, vias 3 -> 2

Commit message: Silkscreen Optimizations
Parts:
- C1: value 1uF -> 0.1uF
- moved R1 1.74 mm to (151.5, 94.7)
- moved SW1 0.36 mm to (140.9, 120.9)
Routing:
- net +3V3: track 39.5 -> 37.4 mm
- net /GPIO18: track 4.31 -> 5.10 mm
Other:
- board text added: "VI"

Commit message: Optimised 4-lyr routing v.4lyr.3
Parts:
- moved R8 1.19 mm to (147.3, 125.0), turned to 270 degrees
- moved R1 0.82 mm to (150.8, 94.2)
- moved R7 0.29 mm to (149.9, 124.3)
Connections:
- D4 pad 4: /GPIO16 -> /GPIO34
Routing:
- net /GPIO16: track 41.7 -> 25.6 mm
- net /GPIO34: track 16.6 -> 31.6 mm, vias 1 -> 2
- net /VI: track 54.6 -> 40.4 mm, vias 3 -> 4
- net GND: track 71.8 -> 63.1 mm, vias 36 -> 37
- net /GPIO8: track 63.4 -> 57.4 mm
- net +3V3: track 37.4 -> 31.6 mm, vias 7 -> 9
- net /CHIP_PU: track 66.6 -> 71.9 mm
- net /RXD0: track 46.4 -> 43.7 mm
- net /GPIO18: track 5.10 -> 2.80 mm, vias 2 -> 0
- net /DN1: track 28.8 -> 31.0 mm
- net /GPIO0: track 75.5 -> 73.7 mm
- net /TXD0: track 47.8 -> 46.1 mm, vias 1 -> 2
- net /GPIO11: track 14.6 -> 16.2 mm
- net /DP1: track 31.3 -> 32.8 mm
- net +BATT: track 6.58 -> 7.86 mm
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- added copper zone on PWR, net /VI

Commit message: minor changes to v.4lyr.3
Routing:
- net GND: track 63.1 -> 64.4 mm
Other:
- board size 27.8 x 70.3 mm -> 27.9 x 68.4 mm
- board text added: "+"
- board text added: "5"
